File: pcb/ahm-panel-placed.kicad_pcb (KiCad board)
At the start: 2 copper layers, 162 x 82 mm, 81 parts, among them J1 UEXT 2x5 box header, J2 JST XH 2-pin, SW1 6x6 mm tact, 5 mm high, SW2 6x6 mm tact, 5 mm high, SW3 6x6 mm tact, 5 mm high, SW4 6x6 mm tact, 5 mm high, U1 MCP23017-E/SO, U2 74AHCT1G125

Commit message: PCB: button LEDs now 5050 WS2812B, re-routed
The WS2812B-2020 footprint was wired with the 5050 pin order (wrong for the
2020 part), and JLCPCB had almost none in stock. All 52 LEDs are now the same
5050 part. Adds export.sh for the production files.

Co-Authored-By: Claude Opus 5.5 (1M context) <noreply@anthropic.com>
Claude-Session: https://claude.ai/code/session_01VPESywWKp5d8Boox5CGCGB
Parts:
- LED49, LED50, LED51, LED52: value WS2812B-2020 -> WS2812B-B; footprint LED_WS2812B-2020_PLCC4_2.0x2.0mm -> LED_WS2812B_PLCC4_5.0x5.0mm_P3.2mm
- moved LED49 1.10 mm to (145.0, 61.5)
- moved LED50 1.10 mm to (105.0, 61.5)
- moved LED51 1.10 mm to (65.0, 61.5)
- moved LED52 1.10 mm to (25.0, 61.5)
