File: pcb/ahm-panel-placed.kicad_pcb (KiCad board)
At the start: 2 copper layers, 162 x 82 mm, 81 parts, among them J1 UEXT 2x5 box header, J2 JST XH 2-pin, SW1 6x6 mm tact, 5 mm high, SW2 6x6 mm tact, 5 mm high, SW3 6x6 mm tact, 5 mm high, SW4 6x6 mm tact, 5 mm high, U1 MCP23017-E/SO, U2 74AHCT1G125

Commit message: PCB review fixes: scene ladder for the Olimex diode, decoupling, power cap
- The Olimex feeds UEXT pin 4 to GPIO36 through a Schottky diode with its own
  10k pull-up (Rev L schematic). With the board's own pull-up the ladder read
  about 0.4 V too high and DJ/IPAD would be confused. Dropped R1, ladder is now
  0/3.3k/8.2k/22k with PCB-specific thresholds in the firmware.
- Dropped the 4.7k I2C pull-ups (the Olimex has 2.2k).
- MCP23017 decoupling cap moved under VDD/VSS (was 16 mm away); re-routed.
- LED brightness capped at 160 to stay well inside the Olimex 5 V / 2 A rail.

Co-Authored-By: Claude Opus 5.5 (1M context) <noreply@anthropic.com>
Claude-Session: https://claude.ai/code/session_01VPESywWKp5d8Boox5CGCGB
Parts:
- removed R1: 10k, R_0805_2012Metric
- removed R6, R7: 4.7k, R_0805_2012Metric
- R2: value 2.2k -> 3.3k
- R3: value 4.7k -> 8.2k
- R4: value 10k -> 22k
- moved C2 15.7 mm to (87.5, 84.4)
- moved U1 2.00 mm to (85.0, 77.0)
