File: pcb/ahm-panel.kicad_pcb (KiCad board)
At the start: 2 copper layers, 162 x 82 mm, 81 parts, among them J1 UEXT 2x5 box header, J2 JST XH 2-pin, SW1 6x6 mm tact, 5 mm high, SW2 6x6 mm tact, 5 mm high, SW3 6x6 mm tact, 5 mm high, SW4 6x6 mm tact, 5 mm high, U1 MCP23017-E/SO, U2 74AHCT1G125

Commit message: PCB: button LEDs now 5050 WS2812B, re-routed
The WS2812B-2020 footprint was wired with the 5050 pin order (wrong for the
2020 part), and JLCPCB had almost none in stock. All 52 LEDs are now the same
5050 part. Adds export.sh for the production files.

Co-Authored-By: Claude Opus 5.5 (1M context) <noreply@anthropic.com>
Claude-Session: https://claude.ai/code/session_01VPESywWKp5d8Boox5CGCGB
Parts:
- LED49, LED50, LED51, LED52: value WS2812B-2020 -> WS2812B-B; footprint LED_WS2812B-2020_PLCC4_2.0x2.0mm -> LED_WS2812B_PLCC4_5.0x5.0mm_P3.2mm
- moved LED49 1.10 mm to (145.0, 61.5)
- moved LED50 1.10 mm to (105.0, 61.5)
- moved LED51 1.10 mm to (65.0, 61.5)
- moved LED52 1.10 mm to (25.0, 61.5)
Routing:
- net LED_5V: track 26.6 -> 7.27 mm
- net SCL: track 63.9 -> 77.3 mm
- net ENC3_SW: track 68.1 -> 79.9 mm, vias 0 -> 1
- net LADDER: track 174.3 -> 163.8 mm
- net ENC4_SW: track 114.7 -> 104.5 mm
- net ENC2_SW: track 66.2 -> 56.4 mm, vias 1 -> 0
- net ENC1_A: track 115.0 -> 106.5 mm
- net ENC2_A: track 72.7 -> 65.4 mm
- net ENC3_A: track 65.8 -> 58.7 mm
- net D28: track 11.2 -> 5.55 mm
- net D18: track 5.37 -> 10.3 mm, vias 0 -> 2
- net D36: track 43.2 -> 47.8 mm
- net D51: track 42.5 -> 38.1 mm
- net ENC3_B: track 56.3 -> 60.4 mm
- net D32: track 8.91 -> 5.32 mm
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